File: pcb/_saved_smartbed.sch (KiCad schematic (older format))
At the start: 53 parts, among them J1 USB_MICRO_A, J2 SBBUS_1, J3 DBGCON, J4 GPIOCON, J5 GPIOCON, J6 FSRCON1, J7 FSRCON2, J8 SBBUS_2, SW1 SW_SPST, U1 LD1117S33CTR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

Commit message: Biggest part of board done
Parts:
- C1, C10, C11, C12, C2, C3, C4, C5, C6, C7, C8, C9: footprint Capacitors_SMD:C_0805_HandSoldering -> Capacitors_SMD:C_0603_HandSoldering
Changed lines of the file:
@@
 F 0 "C8" H 2575 3450 50  0000 L CNN
 F 1 "10uF" H 2575 3250 50  0000 L CNN
-F 2 "Capacitors_SMD:C_0805_HandSoldering" H 2588 3200 50  0001 C CNN
+F 2 "Capacitors_SMD:C_0603_HandSoldering" H 2588 3200 50  0001 C CNN
 F 3 "" H 2550 3350 50  0001 C CNN
 	1    2550 3350
@@
 F 0 "C1" H 1275 3450 50  0000 L CNN
 F 1 "100nF" H 1275 3250 50  0000 L CNN
-F 2 "Capacitors_SMD:C_0805_HandSoldering" H 1288 3200 50  0001 C CNN
+F 2 "Capacitors_SMD:C_0603_HandSoldering" H 1288 3200 50  0001 C CNN
 F 3 "" H 1250 3350 50  0001 C CNN
 	1    1250 3350
@@
 F 0 "C2" H 1425 4850 50  0000 L CNN
 F 1 "6.8pF" H 1425 4650 50  0000 L CNN
-F 2 "Capacitors_SMD:C_0805_HandSoldering" H 1438 4600 50  0001 C CNN
+F 2 "Capacitors_SMD:C_0603_HandSoldering" H 1438 4600 50  0001 C CNN
 F 3 "" H 1400 4750 50  0001 C CNN
 	1    1400 4750
@@
 F 0 "C6" H 2475 4850 50  0000 L CNN
 F 1 "6.8pF" H 2475 4650 50  0000 L CNN
-F 2 "Capacitors_SMD:C_0805_HandSoldering" H 2488 4600 50  0001 C CNN
+F 2 "Capacitors_SMD:C_0603_HandSoldering" H 2488 4600 50  0001 C CNN
 F 3 "" H 2450 4750 50  0001 C CNN
 	1    2450 4750
@@
 F 0 "C4" V 2350 6800 50  0000 L CNN
 F 1 "100nF" V 2050 6700 50  0000 L CNN
-F 2 "Capacitors_SMD:C_0805_HandSoldering" H 2238 6650 50  0001 C CNN
+F 2 "Capacitors_SMD:C_0603_HandSoldering" H 2238 6650 50  0001 C CNN
 F 3 "" H 2200 6800 50  0001 C CNN
 	1    2200 6800
@@
 F 0 "C12" H 9100 2000 50  0000 L CNN
 F 1 "100nF" H 9050 2200 50  0000 L CNN
-F 2 "Capacitors_SMD:C_0805_HandSoldering" H 9088 1950 50  0001 C CNN
+F 2 "Capacitors_SMD:C_0603_HandSoldering" H 9088 1950 50  0001 C CNN
 F 3 "" H 9050 2100 50  0001 C CNN
 	1    9050 2100
@@
 F 0 "C11" H 6725 5350 50  0000 L CNN
 F 1 "100nF" H 6725 5150 50  0000 L CNN
-F 2 "Capacitors_SMD:C_0805_HandSoldering" H 6738 5100 50  0001 C CNN
+F 2 "Capacitors_SMD:C_0603_HandSoldering" H 6738 5100 50  0001 C CNN
 F 3 "" H 6700 5250 50  0001 C CNN
 	1    6700 5250
@@
 F 0 "C7" H 2525 9950 50  0000 L CNN
 F 1 "100nF" H 2525 9750 50  0000 L CNN
-F 2 "Capacitors_SMD:C_0805_HandSoldering" H 2538 9700 50  0001 C CNN
+F 2 "Capacitors_SMD:C_0603_HandSoldering" H 2538 9700 50  0001 C CNN
 F 3 "" H 2500 9850 50  0001 C CNN
 	1    2500 9850
@@
 F 0 "C5" H 2225 9950 50  0000 L CNN
 F 1 "100nF" H 2225 9750 50  0000 L CNN
-F 2 "Capacitors_SMD:C_0805_HandSoldering" H 2238 9700 50  0001 C CNN
+F 2 "Capacitors_SMD:C_0603_HandSoldering" H 2238 9700 50  0001 C CNN
 F 3 "" H 2200 9850 50  0001 C CNN
 	1    2200 9850
@@
 F 0 "C10" H 3125 9950 50  0000 L CNN
 F 1 "100nF" H 3125 9750 50  0000 L CNN
-F 2 "Capacitors_SMD:C_0805_HandSoldering" H 3138 9700 50  0001 C CNN
+F 2 "Capacitors_SMD:C_0603_HandSoldering" H 3138 9700 50  0001 C CNN
 F 3 "" H 3100 9850 50  0001 C CNN
 	1    3100 9850
@@
 F 0 "C9" H 2825 9950 50  0000 L CNN
 F 1 "100nF" H 2825 9750 50  0000 L CNN
-F 2 "Capacitors_SMD:C_0805_HandSoldering" H 2838 9700 50  0001 C CNN
+F 2 "Capacitors_SMD:C_0603_HandSoldering" H 2838 9700 50  0001 C CNN
 F 3 "" H 2800 9850 50  0001 C CNN
 	1    2800 9850
@@
 F 0 "C3" H 1525 1100 50  0000 L CNN
 F 1 "100nF" H 1525 900 50  0000 L CNN
-F 2 "Capacitors_SMD:C_0805_HandSoldering" H 1538 850 50  0001 C CNN
+F 2 "Capacitors_SMD:C_0603_HandSoldering" H 1538 850 50  0001 C CNN
 F 3 "" H 1500 1000 50  0001 C CNN
 	1    1500 1000
