File: pcb/smartbed.kicad_pcb (KiCad board)
At the start: 2 copper layers, 59.5 x 51.5 mm, 51 parts, among them J1 USB_MICRO_A, J2 SBBUS_1, J3 DBGCON, J6 FSRCON1, J7 FSRCON2, J8 SBBUS_2, SW1 SW_SPST, U1 LD1117S33CTR, U2 ATSAMD21J18A, Y1 Crystal

Commit message: Minor changes to PCB, added HTML BOM
Parts:
- removed JP1: JMP, Pin_Headers:Pin_Header_Straight_1x02_Pitch2.54mm
Connections:
- C2 pad 2: Net-(C2-Pad2) -> GND
- C6 pad 2: Net-(C2-Pad2) -> GND
- J1 pad 5: GND -> Net-(J1-Pad5)
- Y1 pad 1: Net-(JP1-Pad2) -> XOUT
Routing:
- net GND: track 448.8 -> 464.9 mm
- net Net-(JP1-Pad2): track 3.89 -> 0.00 mm
- net XIN: track 19.9 -> 16.3 mm
- net Net-(C2-Pad2): track 1.85 -> 0.00 mm
- net XOUT: track 14.1 -> 15.1 mm
